File: panel-connector.kicad_pcb (KiCad board)
At the start: 2 copper layers, 95.9 x 90.2 mm, 223 parts, among them J1 PC104-8BIT, J10 TEST_1P, J105 MOLEX_FFC-14, J11 TEST_1P, J12 TEST_1P, J13 TEST_1P, J2 PC104PTH, J200 MOLEX_FFC-14, J201 CONN-TAB, J202 CONN-TAB, J203 CONN-TAB, J204 CONN-TAB, J210 MOLEX_FFC-14, J211 CONN-TAB, J212 CONN-TAB, J213 CONN-TAB, J214 CONN-TAB, J220 MOLEX_FFC-14, J221 CONN-TAB, J222 CONN-TAB, J223 CONN-TAB, J224 CONN-TAB, J230 MOLEX_FFC-14, J231 CONN-TAB, J232 CONN-TAB, J233 CONN-TAB, J234 CONN-TAB, J3 PC104PTH, J4 PC104PTH, J5 PC104PTH, J6 OEM719, J7 B3B-XH-A(LF)(SN), J8 TEST_1P, J9 TEST_1P, U100 SPV1040, U110 SPV1040, U120 SPV1040, U130 SPV1040, U140 SPV1040, U150 SPV1040, U160 SPV1040, U170 SPV1040, U200 ADG728, U210 ADG728, U220 ADG728, U230 ADG728

Commit message: added file that should have been in previous commit
Other:
- rule pad_to_mask_clearance: 0.03 -> 0.02
Changed lines of the file:
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@@
 (kicad_pcb (version 4) (host pcbnew 4.0.7-e2-6376~58~ubuntu16.04.1)
   (general
-    (links 473)
+    (links 477)
     (no_connects 8)
     (area 83.114286 22.899999 253.885715 168.15)
@@
     (pad_size 5 5)
     (pad_drill 3.45)
-    (pad_to_mask_clearance 0.03)
+    (pad_to_mask_clearance 0.02)
     (pad_to_paste_clearance -0.03)
     (aux_axis_origin 20 140)
@@
     (descr "8-Lead Plastic Thin Shrink Small Outline (ST)-4.4 mm Body [TSSOP] (see Microchip Packaging Specification 00000049BS.pdf)")
     (tags "SSOP 0.65")
+    (solder_mask_margin 0.02)
     (attr smd)
     (fp_text reference U100 (at 0 2.55 180) (layer B.SilkS) hide
@@
     (descr "8-Lead Plastic Thin Shrink Small Outline (ST)-4.4 mm Body [TSSOP] (see Microchip Packaging Specification 00000049BS.pdf)")
     (tags "SSOP 0.65")
+    (solder_mask_margin 0.02)
     (attr smd)
     (fp_text reference U110 (at 0 2.55 180) (layer B.SilkS) hide
@@
     (descr "8-Lead Plastic Thin Shrink Small Outline (ST)-4.4 mm Body [TSSOP] (see Microchip Packaging Specification 00000049BS.pdf)")
     (tags "SSOP 0.65")
+    (solder_mask_margin 0.02)
     (attr smd)
     (fp_text reference U120 (at 0 2.55) (layer B.SilkS) hide
@@
     (descr "8-Lead Plastic Thin Shrink Small Outline (ST)-4.4 mm Body [TSSOP] (see Microchip Packaging Specification 00000049BS.pdf)")
     (tags "SSOP 0.65")
+    (solder_mask_margin 0.02)
     (attr smd)
     (fp_text reference U130 (at 0 2.55) (layer B.SilkS) hide
@@
     (descr "8-Lead Plastic Thin Shrink Small Outline (ST)-4.4 mm Body [TSSOP] (see Microchip Packaging Specification 00000049BS.pdf)")
     (tags "SSOP 0.65")
+    (solder_mask_margin 0.02)
     (attr smd)
     (fp_text reference U140 (at 0 2.55 90) (layer B.SilkS) hide
@@
     (descr "8-Lead Plastic Thin Shrink Small Outline (ST)-4.4 mm Body [TSSOP] (see Microchip Packaging Specification 00000049BS.pdf)")
     (tags "SSOP 0.65")
+    (solder_mask_margin 0.02)
     (attr smd)
     (fp_text reference U150 (at 0 2.55 90) (layer B.SilkS) hide
@@
     (descr "8-Lead Plastic Thin Shrink Small Outline (ST)-4.4 mm Body [TSSOP] (see Microchip Packaging Specification 00000049BS.pdf)")
     (tags "SSOP 0.65")
+    (solder_mask_margin 0.02)
     (attr smd)
     (fp_text reference U160 (at 0.1998 0.0876 270) (layer B.SilkS) hide
@@
     (descr "8-Lead Plastic Thin Shrink Small Outline (ST)-4.4 mm Body [TSSOP] (see Microchip Packaging Specification 00000049BS.pdf)")
     (tags "SSOP 0.65")
+    (solder_mask_margin 0.02)
     (attr smd)
     (fp_text reference U170 (at 0 2.55 270) (layer B.SilkS) hide
@@
   (module SFUSat:MOLEX_FFC-14 (layer B.Cu)
     (at 193 90 270)
+    (solder_mask_margin 0.02)
     (fp_text reference J200 (at 0.5 -5 270) (layer B.SilkS)
       (effects (font (size 1 1) (thickness 0.15)) (justify mirror))
@@
   (module SFUSat:MOLEX_FFC-14 (layer B.Cu)
     (at 153 63)
+    (solder_mask_margin 0.02)
     (fp_text reference J105 (at -2.25 1.5) (layer B.SilkS)
       (effects (font (size 1 1) (thickness 0.15)) (justify mirror))
@@
   (module SFUSat:MOLEX_FFC-14 (layer B.Cu)
     (at 113 90 90)
+    (solder_mask_margin 0.02)
     (fp_text reference J210 (at 0.3 -4.8 270) (layer B.SilkS)
       (effects (font (size 1 1) (thickness 0.15)) (justify mirror))
@@
   (module SFUSat:MOLEX_FFC-14 (layer B.Cu)
     (at 153 127 180)
+    (solder_mask_margin 0.02)
     (fp_text reference J220 (at 0 -5 180) (layer B.SilkS)
       (effects (font (size 1 1) (thickness 0.15)) (justify mirror))
@@
   (module SFUSat:MOLEX_FFC-14 (layer B.Cu)
     (at 153 53)
+    (solder_mask_margin 0.02)
     (fp_text reference J230 (at 0 2.3) (layer B.SilkS)
       (effects (font (size 1 1) (thickness 0.15)) (justify mirror))
@@
   (module SFUSat:TSSOP-16 (layer B.Cu)
     (at 130.8 93.8)
+    (solder_mask_margin 0.03)
     (fp_text reference U210 (at 3.6 0 90) (layer B.SilkS) hide
       (effects (font (size 1 1) (thickness 0.15)) (justify mirror))
